Commit message: Add wheels

File: robotics/project2/src/my_robot/urdf/my_robot.xacro (robot description, xacro)
@@ -11,5 +11,5 @@
     <inertial>
       <mass value="15.0"/>
-      <origin xyz="0.0 0 0" rpy=" 0 0 0"/>
+      <origin xyz="0.0 0 0" rpy="0 0 0"/>
       <inertia
           ixx="0.1" ixy="0" ixz="0"
@@ -19,5 +19,5 @@
     </inertial>
     <collision name='collision'>
-      <origin xyz="0 0 0" rpy=" 0 0 0"/>
+      <origin xyz="0 0 0" rpy="0 0 0"/>
       <geometry>
         <box size=".4 .2 .1"/>
@@ -25,5 +25,5 @@
     </collision>
     <visual name='chassis_visual'>
-      <origin xyz="0 0 0" rpy=" 0 0 0"/>
+      <origin xyz="0 0 0" rpy="0 0 0"/>
       <geometry>
         <box size=".4 .2 .1"/>
@@ -31,5 +31,5 @@
     </visual>
     <collision name='back_caster_collision'>
-      <origin xyz="-0.15 0 -0.05" rpy=" 0 0 0"/>
+      <origin xyz="-0.15 0 -0.05" rpy="0 0 0"/>
       <geometry>
         <sphere radius="0.0499"/>
@@ -37,5 +37,5 @@
     </collision>
     <visual name='back_caster_visual'>
-      <origin xyz="-0.15 0 -0.05" rpy=" 0 0 0"/>
+      <origin xyz="-0.15 0 -0.05" rpy="0 0 0"/>
       <geometry>
         <sphere radius="0.05"/>
@@ -43,5 +43,5 @@
     </visual>
     <collision name='front_caster_collision'>
-      <origin xyz="0.15 0 -0.05" rpy=" 0 0 0"/>
+      <origin xyz="0.15 0 -0.05" rpy="0 0 0"/>
       <geometry>
         <sphere radius="0.0499"/>
@@ -49,5 +49,5 @@
     </collision>
     <visual name='front_caster_visual'>
-      <origin xyz="0.15 0 -0.05" rpy=" 0 0 0"/>
+      <origin xyz="0.15 0 -0.05" rpy="0 0 0"/>
       <geometry>
         <sphere radius="0.05"/>
@@ -55,3 +55,65 @@
     </visual>
   </link>
+  <link name='left_wheel'>
+    <inertial>
+      <mass value="5.0"/>
+      <origin xyz="0.0 0 0" rpy="0 1.5707 1.5707"/>
+      <inertia
+          ixx="0.1" ixy="0" ixz="0"
+          iyy="0.1" iyz="0"
+          izz="0.1"
+      />
+    </inertial>
+    <collision name='collision'>
+      <origin xyz="0 0 0" rpy="0 1.5707 1.5707"/>
+      <geometry>
+        <cylinder radius=".1" length=".05"/>
+      </geometry>
+    </collision>
+    <visual name='chassis_visual'>
+      <origin xyz="0 0 0" rpy="0 1.5707 1.5707"/>
+      <geometry>
+        <cylinder radius=".1" length=".05"/>
+      </geometry>
+    </visual>
+  </link>
+  <link name='right_wheel'>
+    <inertial>
+      <mass value="5.0"/>
+      <origin xyz="0.0 0 0" rpy="0 1.5707 1.5707"/>
+      <inertia
+          ixx="0.1" ixy="0" ixz="0"
+          iyy="0.1" iyz="0"
+          izz="0.1"
+      />
+    </inertial>
+    <collision name='collision'>
+      <origin xyz="0 0 0" rpy="0 1.5707 1.5707"/>
+      <geometry>
+        <cylinder radius=".1" length=".05"/>
+      </geometry>
+    </collision>
+    <visual name='chassis_visual'>
+      <origin xyz="0 0 0" rpy=" 0 1.5707 1.5707"/>
+      <geometry>
+        <cylinder radius=".1" length=".05"/>
+      </geometry>
+    </visual>
+  </link>
+  <joint type="continuous" name="left_wheel_hinge">
+    <origin xyz="0 0.15 0" rpy="0 0 0"/>
+    <child link="left_wheel"/>
+    <parent link="chassis"/>
+    <axis xyz="0 1 0" rpy="0 0 0"/>
+    <limit effort="10000" velocity="1000"/>
+    <dynamics damping="1.0" friction="1.0"/>
+  </joint>
+  <joint type="continuous" name="right_wheel_hinge">
+    <origin xyz="0 -0.15 0" rpy="0 0 0"/>
+    <child link="right_wheel"/>
+    <parent link="chassis"/>
+    <axis xyz="0 1 0" rpy="0 0 0"/>
+    <limit effort="10000" velocity="1000"/>
+    <dynamics damping="1.0" friction="1.0"/>
+  </joint>
 </robot>

Commit message: Add camera and hokuyo lidar

File: robotics/project2/src/my_robot/urdf/my_robot.xacro (robot description, xacro)
@@ -18,5 +18,5 @@
       />
     </inertial>
-    <collision name='collision'>
+    <collision name='chassis_collision'>
       <origin xyz="0 0 0" rpy="0 0 0"/>
       <geometry>
@@ -65,5 +65,5 @@
       />
     </inertial>
-    <collision name='collision'>
+    <collision name='left_wheel_collision'>
       <origin xyz="0 0 0" rpy="0 1.5707 1.5707"/>
       <geometry>
@@ -71,5 +71,5 @@
       </geometry>
     </collision>
-    <visual name='chassis_visual'>
+    <visual name='left_wheel_collision'>
       <origin xyz="0 0 0" rpy="0 1.5707 1.5707"/>
       <geometry>
@@ -88,5 +88,5 @@
       />
     </inertial>
-    <collision name='collision'>
+    <collision name='right_wheel_collision'>
       <origin xyz="0 0 0" rpy="0 1.5707 1.5707"/>
       <geometry>
@@ -94,5 +94,5 @@
       </geometry>
     </collision>
-    <visual name='chassis_visual'>
+    <visual name='right_wheel_visual'>
       <origin xyz="0 0 0" rpy=" 0 1.5707 1.5707"/>
       <geometry>
@@ -117,3 +117,62 @@
     <dynamics damping="1.0" friction="1.0"/>
   </joint>
+  <link name='camera'>
+    <box_inertia m="0.1" w="0.05" h="0.05" d="0.05"/>
+    <inertial>
+      <mass value="0.1"/>
+      <origin xyz="0 0 0" rpy="0 0 0"/>
+      <inertia
+          ixx="1e-6" ixy="0" ixz="0"
+          iyy="1e-6" iyz="0"
+          izz="1e-6"
+      />
+    </inertial>
+    <collision name='camera_collision'>
+      <origin xyz="0 0 0" rpy="0 0 0"/>
+      <geometry>
+        <box size=".05 .05 .05"/>
+      </geometry>
+    </collision>
+    <visual name='camera_visual'>
+      <origin xyz="0 0 0" rpy="0 0 0"/>
+      <geometry>
+        <box size=".05 .05 .05"/>
+      </geometry>
+    </visual>
+  </link>
+  <joint type="fixed" name="camera_joint">
+    <origin xyz="0.2 0 0" rpy="0 0 0"/>
+    <child link="camera"/>
+    <parent link="chassis"/>
+    <axis xyz="0 1 0"/>
+  </joint>
+  <link name='hokuyo'>
+    <inertial>
+      <mass value="1e-5"/>
+      <origin xyz="0 0 0" rpy="0 0 0"/>
+      <inertia
+          ixx="1e-6" ixy="0" ixz="0"
+          iyy="1e-6" iyz="0"
+          izz="1e-6"
+      />
+    </inertial>
+    <collision name='hokuyo_collision'>
+      <origin xyz="0 0 0" rpy="0 0 0"/>
+      <geometry>
+        <box size=".1 .1 .1"/>
+      </geometry>
+    </collision>
+    <visual name='hokuyo_visual'>
+      <origin xyz="0 0 0" rpy="0 0 0"/>
+      <geometry>
+        <mesh filename="package://my_robot/meshes/hokuyo.dae"/>
+      </geometry>
+    </visual>
+  </link>
+  <joint type="fixed" name="hokuyo_joint">
+    <origin xyz="0.15 0 .1" rpy="0 0 0"/>
+    <child link="hokuyo"/>
+    <parent link="chassis"/>
+    <axis xyz="0 1 0"/>
+  </joint>
 </robot>

Commit message: Update robot shape

File: robotics/project2/src/my_robot/urdf/my_robot.xacro (robot description, xacro)
@@ -9,5 +9,5 @@
   </joint>
   <link name='chassis'>
-    <pose>0 0 0.1 0 0 0</pose>
+    <pose>0 0 0.2 0 0 0</pose>
     <inertial>
       <mass value="15.0"/>
@@ -22,5 +22,5 @@
       <origin xyz="0 0 0" rpy="0 0 0"/>
       <geometry>
-        <box size=".4 .2 .1"/>
+        <box size=".5 .1 .2"/>
       </geometry>
     </collision>
@@ -28,29 +28,29 @@
       <origin xyz="0 0 0" rpy="0 0 0"/>
       <geometry>
-        <box size=".4 .2 .1"/>
+        <box size=".5 .1 .2"/>
+      </geometry>
+    </visual>
+    <collision name='tower_collision'>
+      <origin xyz=".2 0 .2" rpy="0 0 0"/>
+      <geometry>
+        <box size=".1 .1 .2"/>
+      </geometry>
+    </collision>
+    <visual name='tower_visual'>
+      <origin xyz=".2 0 .2" rpy="0 0 0"/>
+      <geometry>
+        <box size=".1 .1 .2"/>
       </geometry>
     </visual>
     <collision name='back_caster_collision'>
-      <origin xyz="-0.15 0 -0.05" rpy="0 0 0"/>
+      <origin xyz="-0.2 0 -0.1" rpy="0 0 0"/>
       <geometry>
-        <sphere radius="0.0499"/>
+        <sphere radius="0.0999"/>
       </geometry>
     </collision>
     <visual name='back_caster_visual'>
-      <origin xyz="-0.15 0 -0.05" rpy="0 0 0"/>
+      <origin xyz="-0.2 0 -0.1" rpy="0 0 0"/>
       <geometry>
-        <sphere radius="0.05"/>
-      </geometry>
-    </visual>
-    <collision name='front_caster_collision'>
-      <origin xyz="0.15 0 -0.05" rpy="0 0 0"/>
-      <geometry>
-        <sphere radius="0.0499"/>
-      </geometry>
-    </collision>
-    <visual name='front_caster_visual'>
-      <origin xyz="0.15 0 -0.05" rpy="0 0 0"/>
-      <geometry>
-        <sphere radius="0.05"/>
+        <sphere radius="0.1"/>
       </geometry>
     </visual>
@@ -69,5 +69,5 @@
       <origin xyz="0 0 0" rpy="0 1.5707 1.5707"/>
       <geometry>
-        <cylinder radius=".1" length=".05"/>
+        <cylinder radius=".2" length=".075"/>
       </geometry>
     </collision>
@@ -75,5 +75,5 @@
       <origin xyz="0 0 0" rpy="0 1.5707 1.5707"/>
       <geometry>
-        <cylinder radius=".1" length=".05"/>
+        <cylinder radius=".2" length=".075"/>
       </geometry>
     </visual>
@@ -92,5 +92,5 @@
       <origin xyz="0 0 0" rpy="0 1.5707 1.5707"/>
       <geometry>
-        <cylinder radius=".1" length=".05"/>
+        <cylinder radius=".2" length=".075"/>
       </geometry>
     </collision>
@@ -98,10 +98,10 @@
       <origin xyz="0 0 0" rpy=" 0 1.5707 1.5707"/>
       <geometry>
-        <cylinder radius=".1" length=".05"/>
+        <cylinder radius=".2" length=".075"/>
       </geometry>
     </visual>
   </link>
   <joint type="continuous" name="left_wheel_hinge">
-    <origin xyz="0 0.15 0" rpy="0 0 0"/>
+    <origin xyz="0.15 0.1 0" rpy="0 0 0"/>
     <child link="left_wheel"/>
     <parent link="chassis"/>
@@ -111,5 +111,5 @@
   </joint>
   <joint type="continuous" name="right_wheel_hinge">
-    <origin xyz="0 -0.15 0" rpy="0 0 0"/>
+    <origin xyz="0.15 -0.1 0" rpy="0 0 0"/>
     <child link="right_wheel"/>
     <parent link="chassis"/>
@@ -143,5 +143,5 @@
   </link>
   <joint type="fixed" name="camera_joint">
-    <origin xyz="0.2 0 0" rpy="0 0 0"/>
+    <origin xyz="0.275 0 .2" rpy="0 0 0"/>
     <child link="camera"/>
     <parent link="chassis"/>
@@ -172,5 +172,5 @@
   </link>
   <joint type="fixed" name="hokuyo_joint">
-    <origin xyz="0.15 0 .1" rpy="0 0 0"/>
+    <origin xyz="0.3 0 .1" rpy="0 0 0"/>
     <child link="hokuyo"/>
     <parent link="chassis"/>

Commit message: Material colors

File: robotics/project2/src/my_robot/urdf/my_robot.xacro (robot description, xacro)
@@ -2,4 +2,10 @@
 <robot name="my_robot" xmlns:xacro="http://www.ros.org/wiki/xacro">
   <xacro:include filename="$(find my_robot)/urdf/my_robot.gazebo" />
+  <material name="greenish">
+      <color rgba="0 .8 0.2 1"/>
+  </material>
+  <material name="dark">
+      <color rgba="0.05 .05 0.05 1"/>
+  </material>
   <link name="robot_footprint"></link>
   <joint name="robot_footprint_joint" type="fixed">
@@ -30,4 +36,5 @@
         <box size=".5 .1 .2"/>
       </geometry>
+      <material name="greenish"/>
     </visual>
     <collision name='tower_collision'>
@@ -42,4 +49,5 @@
         <box size=".1 .1 .2"/>
       </geometry>
+      <material name="greenish"/>
     </visual>
     <collision name='back_caster_collision'>
@@ -72,9 +80,10 @@
       </geometry>
     </collision>
-    <visual name='left_wheel_collision'>
+    <visual name='left_wheel_visual'>
       <origin xyz="0 0 0" rpy="0 1.5707 1.5707"/>
       <geometry>
         <cylinder radius=".2" length=".075"/>
       </geometry>
+      <material name="dark"/>
     </visual>
   </link>
@@ -100,4 +109,5 @@
         <cylinder radius=".2" length=".075"/>
       </geometry>
+      <material name="dark"/>
     </visual>
   </link>

Commit message: Change shape

File: robotics/project2/src/my_robot/urdf/my_robot.xacro (robot description, xacro)
@@ -39,13 +39,13 @@
     </visual>
     <collision name='tower_collision'>
-      <origin xyz=".2 0 .2" rpy="0 0 0"/>
+      <origin xyz=".3 0 .2" rpy="0 0 0"/>
       <geometry>
-        <box size=".1 .1 .2"/>
+        <box size=".3 .1 .2"/>
       </geometry>
     </collision>
     <visual name='tower_visual'>
-      <origin xyz=".2 0 .2" rpy="0 0 0"/>
+      <origin xyz=".3 0 .2" rpy="0 0 0"/>
       <geometry>
-        <box size=".1 .1 .2"/>
+        <box size=".3 .1 .2"/>
       </geometry>
       <material name="greenish"/>
@@ -153,5 +153,5 @@
   </link>
   <joint type="fixed" name="camera_joint">
-    <origin xyz="0.275 0 .2" rpy="0 0 0"/>
+    <origin xyz="0.475 0 .2" rpy="0 0 0"/>
     <child link="camera"/>
     <parent link="chassis"/>
@@ -182,5 +182,5 @@
   </link>
   <joint type="fixed" name="hokuyo_joint">
-    <origin xyz="0.3 0 .1" rpy="0 0 0"/>
+    <origin xyz="0.5 0 .1" rpy="0 0 0"/>
     <child link="hokuyo"/>
     <parent link="chassis"/>

Commit message: Change shape again

File: robotics/project2/src/my_robot/urdf/my_robot.xacro (robot description, xacro)
@@ -3,8 +3,8 @@
   <xacro:include filename="$(find my_robot)/urdf/my_robot.gazebo" />
   <material name="greenish">
-      <color rgba="0 .8 0.2 1"/>
+      <color rgba="0.0 0.8 0.2 1"/>
   </material>
   <material name="dark">
-      <color rgba="0.05 .05 0.05 1"/>
+      <color rgba="0.05 0.05 0.05 1"/>
   </material>
   <link name="robot_footprint"></link>
@@ -39,13 +39,13 @@
     </visual>
     <collision name='tower_collision'>
-      <origin xyz=".3 0 .2" rpy="0 0 0"/>
+      <origin xyz=".25 0 .2" rpy="0 0 0"/>
       <geometry>
-        <box size=".3 .1 .2"/>
+        <box size=".1 .1 .2"/>
       </geometry>
     </collision>
     <visual name='tower_visual'>
-      <origin xyz=".3 0 .2" rpy="0 0 0"/>
+      <origin xyz=".25 0 .2" rpy="0 0 0"/>
       <geometry>
-        <box size=".3 .1 .2"/>
+        <box size=".1 .1 .2"/>
       </geometry>
       <material name="greenish"/>
@@ -77,5 +77,5 @@
       <origin xyz="0 0 0" rpy="0 1.5707 1.5707"/>
       <geometry>
-        <cylinder radius=".2" length=".075"/>
+        <cylinder radius=".075" length=".025"/>
       </geometry>
     </collision>
@@ -83,5 +83,5 @@
       <origin xyz="0 0 0" rpy="0 1.5707 1.5707"/>
       <geometry>
-        <cylinder radius=".2" length=".075"/>
+        <cylinder radius=".075" length=".025"/>
       </geometry>
       <material name="dark"/>
@@ -101,5 +101,5 @@
       <origin xyz="0 0 0" rpy="0 1.5707 1.5707"/>
       <geometry>
-        <cylinder radius=".2" length=".075"/>
+        <cylinder radius=".075" length=".025"/>
       </geometry>
     </collision>
@@ -107,5 +107,5 @@
       <origin xyz="0 0 0" rpy=" 0 1.5707 1.5707"/>
       <geometry>
-        <cylinder radius=".2" length=".075"/>
+        <cylinder radius=".075" length=".025"/>
       </geometry>
       <material name="dark"/>
@@ -113,5 +113,5 @@
   </link>
   <joint type="continuous" name="left_wheel_hinge">
-    <origin xyz="0.15 0.1 0" rpy="0 0 0"/>
+    <origin xyz="0.15 0.1 -0.075" rpy="0 0 0"/>
     <child link="left_wheel"/>
     <parent link="chassis"/>
@@ -121,5 +121,5 @@
   </joint>
   <joint type="continuous" name="right_wheel_hinge">
-    <origin xyz="0.15 -0.1 0" rpy="0 0 0"/>
+    <origin xyz="0.15 -0.1 -.075" rpy="0 0 0"/>
     <child link="right_wheel"/>
     <parent link="chassis"/>
@@ -153,5 +153,5 @@
   </link>
   <joint type="fixed" name="camera_joint">
-    <origin xyz="0.475 0 .2" rpy="0 0 0"/>
+    <origin xyz="0.275 0 .2" rpy="0 0 0"/>
     <child link="camera"/>
     <parent link="chassis"/>
@@ -182,5 +182,5 @@
   </link>
   <joint type="fixed" name="hokuyo_joint">
-    <origin xyz="0.5 0 .1" rpy="0 0 0"/>
+    <origin xyz="0.3 0 .1" rpy="0 0 0"/>
     <child link="hokuyo"/>
     <parent link="chassis"/>

Commit message: Fix color

File: robotics/project2/src/my_robot/urdf/my_robot.xacro (robot description, xacro)
@@ -36,8 +36,7 @@
         <box size=".5 .1 .2"/>
       </geometry>
-      <material name="greenish"/>
     </visual>
     <collision name='tower_collision'>
-      <origin xyz=".25 0 .2" rpy="0 0 0"/>
+      <origin xyz=".2 0 .2" rpy="0 0 0"/>
       <geometry>
         <box size=".1 .1 .2"/>
@@ -45,5 +44,5 @@
     </collision>
     <visual name='tower_visual'>
-      <origin xyz=".25 0 .2" rpy="0 0 0"/>
+      <origin xyz=".2 0 .2" rpy="0 0 0"/>
       <geometry>
         <box size=".1 .1 .2"/>
@@ -54,5 +53,5 @@
       <origin xyz="-0.2 0 -0.1" rpy="0 0 0"/>
       <geometry>
-        <sphere radius="0.0999"/>
+        <sphere radius="0.0499"/>
       </geometry>
     </collision>
@@ -60,5 +59,5 @@
       <origin xyz="-0.2 0 -0.1" rpy="0 0 0"/>
       <geometry>
-        <sphere radius="0.1"/>
+        <sphere radius="0.5"/>
       </geometry>
     </visual>
@@ -153,5 +152,5 @@
   </link>
   <joint type="fixed" name="camera_joint">
-    <origin xyz="0.275 0 .2" rpy="0 0 0"/>
+    <origin xyz="0.275 0 0" rpy="0 0 0"/>
     <child link="camera"/>
     <parent link="chassis"/>
@@ -182,5 +181,5 @@
   </link>
   <joint type="fixed" name="hokuyo_joint">
-    <origin xyz="0.3 0 .1" rpy="0 0 0"/>
+    <origin xyz="0.3 0 .1" rpy="0 0 0.2"/>
     <child link="hokuyo"/>
     <parent link="chassis"/>

Commit message: Fix bug

File: robotics/project2/src/my_robot/urdf/my_robot.xacro (robot description, xacro)
@@ -59,5 +59,5 @@
       <origin xyz="-0.2 0 -0.1" rpy="0 0 0"/>
       <geometry>
-        <sphere radius="0.5"/>
+        <sphere radius="0.05"/>
       </geometry>
     </visual>

Commit message: More colors

File: robotics/project2/src/my_robot/urdf/my_robot.xacro (robot description, xacro)
@@ -2,10 +2,4 @@
 <robot name="my_robot" xmlns:xacro="http://www.ros.org/wiki/xacro">
   <xacro:include filename="$(find my_robot)/urdf/my_robot.gazebo" />
-  <material name="greenish">
-      <color rgba="0.0 0.8 0.2 1"/>
-  </material>
-  <material name="dark">
-      <color rgba="0.05 0.05 0.05 1"/>
-  </material>
   <link name="robot_footprint"></link>
   <joint name="robot_footprint_joint" type="fixed">
@@ -48,5 +42,4 @@
         <box size=".1 .1 .2"/>
       </geometry>
-      <material name="greenish"/>
     </visual>
     <collision name='back_caster_collision'>
@@ -84,5 +77,4 @@
         <cylinder radius=".075" length=".025"/>
       </geometry>
-      <material name="dark"/>
     </visual>
   </link>
@@ -108,5 +100,4 @@
         <cylinder radius=".075" length=".025"/>
       </geometry>
-      <material name="dark"/>
     </visual>
   </link>

Commit message: One more fix

File: robotics/project2/src/my_robot/urdf/my_robot.xacro (robot description, xacro)
@@ -103,5 +103,5 @@
   </link>
   <joint type="continuous" name="left_wheel_hinge">
-    <origin xyz="0.15 0.1 -0.075" rpy="0 0 0"/>
+    <origin xyz="0.15 0.075 -0.075" rpy="0 0 0"/>
     <child link="left_wheel"/>
     <parent link="chassis"/>
@@ -111,5 +111,5 @@
   </joint>
   <joint type="continuous" name="right_wheel_hinge">
-    <origin xyz="0.15 -0.1 -.075" rpy="0 0 0"/>
+    <origin xyz="0.15 -0.075 -.075" rpy="0 0 0"/>
     <child link="right_wheel"/>
     <parent link="chassis"/>
@@ -143,5 +143,5 @@
   </link>
   <joint type="fixed" name="camera_joint">
-    <origin xyz="0.275 0 0" rpy="0 0 0"/>
+    <origin xyz="0.275 0 -.05" rpy="0 0 0"/>
     <child link="camera"/>
     <parent link="chassis"/>
@@ -172,5 +172,5 @@
   </link>
   <joint type="fixed" name="hokuyo_joint">
-    <origin xyz="0.3 0 .1" rpy="0 0 0.2"/>
+    <origin xyz="0.225 0 .35" rpy="0 0 0"/>
     <child link="hokuyo"/>
     <parent link="chassis"/>

Commit message: Move to front

File: robotics/project2/src/my_robot/urdf/my_robot.xacro (robot description, xacro)
@@ -172,5 +172,5 @@
   </link>
   <joint type="fixed" name="hokuyo_joint">
-    <origin xyz="0.225 0 .35" rpy="0 0 0"/>
+    <origin xyz="0.275 0 .3" rpy="0 0 0"/>
     <child link="hokuyo"/>
     <parent link="chassis"/>

Commit message: Move caster

File: robotics/project2/src/my_robot/urdf/my_robot.xacro (robot description, xacro)
@@ -44,5 +44,5 @@
     </visual>
     <collision name='back_caster_collision'>
-      <origin xyz="-0.2 0 -0.1" rpy="0 0 0"/>
+      <origin xyz="-0.05 0 -0.1" rpy="0 0 0"/>
       <geometry>
         <sphere radius="0.0499"/>
@@ -50,5 +50,5 @@
     </collision>
     <visual name='back_caster_visual'>
-      <origin xyz="-0.2 0 -0.1" rpy="0 0 0"/>
+      <origin xyz="-0.05 0 -0.1" rpy="0 0 0"/>
       <geometry>
         <sphere radius="0.05"/>
